Commit message: URDF wheel axis 4

File: jainbot/urdf/jainbot.urdf.xacro (robot description, xacro)
@@ -96,5 +96,5 @@
     <child  link="left_wheel"/>
     <origin xyz="0.135 -0.195 -0.055" rpy="0 0 0"/>
-    <axis xyz="0 -1 0"/>
+    <axis xyz="0 1 0"/>
   </joint>
   <joint name="right_wheel_joint" type="continuous">
@@ -102,5 +102,5 @@
     <child  link="right_wheel"/>
     <origin xyz="0.135 0.195 -0.055" rpy="0 0 0"/>
-    <axis xyz="0 -1 0"/>
+    <axis xyz="0 1 0"/>
   </joint>
   <!-- ===== Casters (visual-only) ===== -->

Commit message: URDF chassis axis fix

File: jainbot/urdf/jainbot.urdf.xacro (robot description, xacro)
@@ -8,6 +8,6 @@
        Wheel separation: 0.390 => y = +/- 0.195
        Wheels are 0.110 from rear edge:
-         rear edge x = +0.245 (chassis centered)
-         wheel x = +0.245 - 0.110 = +0.135
+         rear edge x = -0.245 (chassis centered)
+         wheel x = -0.245 + 0.110 = -0.135
        Wheels ~0.050 below chassis bottom.
        Chassis base plate thickness: 0.010 (just for RViz visuals)
@@ -95,5 +95,5 @@
     <parent link="base_link"/>
     <child  link="left_wheel"/>
-    <origin xyz="0.135 -0.195 -0.055" rpy="0 0 0"/>
+    <origin xyz="-0.135 0.195 -0.055" rpy="0 0 0"/>
     <axis xyz="0 1 0"/>
   </joint>
@@ -101,5 +101,5 @@
     <parent link="base_link"/>
     <child  link="right_wheel"/>
-    <origin xyz="0.135 0.195 -0.055" rpy="0 0 0"/>
+    <origin xyz="-0.135 -0.195 -0.055" rpy="0 0 0"/>
     <axis xyz="0 1 0"/>
   </joint>
@@ -125,5 +125,5 @@
     </visual>
   </link>
-  <!-- Casters: x=-0.145, y=+/-0.0825; put them near ground -->
+  <!-- Casters: x=+0.145, y=+/-0.0825; put them near ground -->
   <!-- wheel ground contact is at z = -0.1075 in base_link frame -->
   <!-- caster center z = -0.1075 + 0.020 = -0.0875 -->
@@ -131,10 +131,10 @@
     <parent link="base_link"/>
     <child link="caster_left"/>
-    <origin xyz="-0.145 -0.0825 -0.0875" rpy="0 0 0"/>
+    <origin xyz="0.145 0.0825 -0.0875" rpy="0 0 0"/>
   </joint>
   <joint name="caster_right_joint" type="fixed">
     <parent link="base_link"/>
     <child link="caster_right"/>
-    <origin xyz="-0.145 0.0825 -0.0875" rpy="0 0 0"/>
+    <origin xyz="0.145 -0.0825 -0.0875" rpy="0 0 0"/>
   </joint>
   <!-- ===== IMU (visual-only link, useful for TF) ===== -->
@@ -149,10 +149,10 @@
     </visual>
   </link>
-  <!-- IMU: 60mm from front => x=-0.185, 175mm from sides => basically centerline (y=0) -->
+  <!-- IMU: 60mm from front => x=+0.185, 175mm from sides => basically centerline (y=0) -->
   <joint name="imu_joint" type="fixed">
     <parent link="base_link"/>
     <child link="imu_link"/>
     <!-- place it slightly above chassis center so it appears on top -->
-    <origin xyz="-0.185 0.0 0.0" rpy="0 3.14159265359 0"/>
+    <origin xyz="0.185 0.0 0.0" rpy="0 3.14159265359 0"/>
   </joint>
   <!-- =========================

Commit message: URDF axis fix

File: jainbot/urdf/jainbot.urdf.xacro (robot description, xacro)
@@ -95,12 +95,12 @@
     <parent link="base_link"/>
     <child  link="left_wheel"/>
-    <origin xyz="-0.135 0.195 -0.055" rpy="0 0 0"/>
-    <axis xyz="0 1 0"/>
+    <origin xyz="-0.135 -0.195 -0.055" rpy="0 0 0"/>
+    <axis xyz="0 -1 0"/>
   </joint>
   <joint name="right_wheel_joint" type="continuous">
     <parent link="base_link"/>
     <child  link="right_wheel"/>
-    <origin xyz="-0.135 -0.195 -0.055" rpy="0 0 0"/>
-    <axis xyz="0 1 0"/>
+    <origin xyz="-0.135 0.195 -0.055" rpy="0 0 0"/>
+    <axis xyz="0 -1 0"/>
   </joint>
   <!-- ===== Casters (visual-only) ===== -->
@@ -131,10 +131,10 @@
     <parent link="base_link"/>
     <child link="caster_left"/>
-    <origin xyz="0.145 0.0825 -0.0875" rpy="0 0 0"/>
+    <origin xyz="0.145 -0.0825 -0.0875" rpy="0 0 0"/>
   </joint>
   <joint name="caster_right_joint" type="fixed">
     <parent link="base_link"/>
     <child link="caster_right"/>
-    <origin xyz="0.145 -0.0825 -0.0875" rpy="0 0 0"/>
+    <origin xyz="0.145 0.0825 -0.0875" rpy="0 0 0"/>
   </joint>
   <!-- ===== IMU (visual-only link, useful for TF) ===== -->

Commit message: camera stuff added to launch file and URDF

File: jainbot/urdf/jainbot.urdf.xacro (robot description, xacro)
@@ -156,4 +156,19 @@
     <!-- place it slightly above chassis center so it appears on top -->
     <origin xyz="0.185 0.0 0.0" rpy="0 3.14159265359 0"/>
+  </joint>
+  <!-- ===== Camera (RealSense D435) ===== -->
+  <link name="camera_link">
+    <visual>
+      <geometry>
+        <box size="0.090 0.025 0.025"/>
+      </geometry>
+      <material name="blue"/>
+    </visual>
+  </link>
+  <!-- Camera: front of chassis, on top of wall -->
+  <joint name="camera_joint" type="fixed">
+    <parent link="base_link"/>
+    <child link="camera_link"/>
+    <origin xyz="0.245 0.0 0.130" rpy="0 0 0"/>
   </joint>
   <!-- =========================
